File: PANS.brd (EAGLE design)
At the start: 68.5 x 109.2 mm, 69 parts, among them IC1 TL074, IC2 TL074, J1 THONKICONNNEW, J15 power, J2 THONKICONNNEW, J3 THONKICONNNEW, J4 THONKICONNNEW, J5 THONKICONNNEW, J6 THONKICONNNEW, J7 Stereo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

Commit message: Add files via upload
Parts:
- removed R18, R19: 1K, resistor:M0805
- PAN: value 10K -> B1M
- moved R21 9.30 mm to (52.5, 38.7), turned to 90 degrees
- moved R20 2.67 mm to (47.5, 38.7), turned to 90 degrees
Connections:
- removed net N$35: J6.P$1_TIP, R18.2, R19.2, VOL.2
- new net N$34: J6.P$1_TIP, PAN.2, VOL.2
- net GND: no longer PAN.2
- net N$36: no longer R19.1
- net N$38: no longer R18.1
Routing:
- net N$34: track 0.00 -> 85.2 mm
- net N$35: track 82.6 -> 0.00 mm
- net N$43: track 68.3 -> 80.8 mm
- net N$36: track 13.4 -> 2.55 mm
- net N$38: track 8.88 -> 2.53 mm
- net N$41: track 62.2 -> 60.1 mm
Changed lines of the file:
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@@
 <drawing>
 <settings>
-<setting alwaysvectorfont="yes"/>
+<setting alwaysvectorfont="no"/>
 <setting verticaltext="up"/>
 </settings>
-<grid distance="0.005" unitdist="inch" unit="inch" style="dots" multiple="1" display="yes" altdistance="5" altunitdist="mil" altunit="mil"/>
+<grid distance="0.01" unitdist="inch" unit="inch" style="dots" multiple="1" display="yes" altdistance="5" altunitdist="mil" altunit="mil"/>
 <layers>
 <layer number="1" name="Top" color="4" fill="1" visible="yes" active="yes"/>
@@
 <attribute name="VALUE" x="17.145" y="31.115" size="1.27" layer="28" rot="MR0"/>
 </element>
-<element name="R18" library="resistor" package="M0805" value="1K" x="50.165" y="35.814" smashed="yes" rot="MR0">
-<attribute name="NAME" x="48.26" y="35.179" size="1.27" layer="26" rot="MR0"/>
-<attribute name="VALUE" x="48.26" y="33.909" size="1.27" layer="28" rot="MR0"/>
-</element>
-<element name="R19" library="resistor" package="M0805" value="1K" x="50.165" y="32.639" smashed="yes" rot="MR0">
-<attribute name="NAME" x="48.26" y="32.004" size="1.27" layer="26" rot="MR0"/>
-<attribute name="VALUE" x="48.26" y="30.734" size="1.27" layer="28" rot="MR0"/>
-</element>
 <element name="R2" library="resistor" package="M0805" value="1K" x="20.955" y="85.09" smashed="yes" rot="MR180">
 <attribute name="NAME" x="23.495" y="85.725" size="1.27" layer="26" rot="MR180"/>
 <attribute name="VALUE" x="16.51" y="85.725" size="1.27" layer="28" rot="MR180"/>
 </element>
-<element name="R20" library="resistor" package="M0805" value="1K" x="50.165" y="38.735" smashed="yes" rot="MR180">
-<attribute name="NAME" x="45.085" y="39.37" size="1.27" layer="26" rot="MR180"/>
-<attribute name="VALUE" x="46.355" y="38.1" size="1.27" layer="28" rot="MR180"/>
-</element>
-<element name="R21" library="resistor" package="M0805" value="1K" x="50.165" y="29.718" smashed="yes" rot="MR180">
-<attribute name="NAME" x="45.085" y="30.353" size="1.27" layer="26" rot="MR180"/>
-<attribute name="VALUE" x="45.085" y="29.083" size="1.27" layer="28" rot="MR180"/>
+<element name="R20" library="resistor" package="M0805" value="1K" x="47.498" y="38.735" smashed="yes" rot="MR90">
+<attribute name="NAME" x="46.863" y="33.655" size="1.27" layer="26" rot="MR90"/>
+<attribute name="VALUE" x="48.133" y="34.925" size="1.27" layer="28" rot="MR90"/>
+</element>
+<element name="R21" library="resistor" package="M0805" value="1K" x="52.451" y="38.735" smashed="yes" rot="MR90">
+<attribute name="NAME" x="51.816" y="33.655" size="1.27" layer="26" rot="MR90"/>
+<attribute name="VALUE" x="53.086" y="33.655" size="1.27" layer="28" rot="MR90"/>
 </element>
 <element name="R22" library="resistor" package="M0805" value="1k" x="40.767" y="61.976" smashed="yes" rot="MR0">
@@
 <attribute name="VALUE" x="22.225" y="51.689" size="1.27" layer="27"/>
 </element>
-<element name="PAN" library="MusicThingModular" package="9MM_SNAP-IN_POT" value="10K" x="50.165" y="49.149" smashed="yes">
+<element name="PAN" library="MusicThingModular" package="9MM_SNAP-IN_POT" value="B1M" x="50.165" y="49.149" smashed="yes">
 <attribute name="NAME" x="46.355" y="51.689" size="1.0668" layer="25"/>
 <attribute name="VALUE" x="51.435" y="51.689" size="1.27" layer="27"/>
@@
 <contactref element="R10" pad="1"/>
 <contactref element="J6" pad="P$3_SLEEVE"/>
-<contactref element="PAN" pad="2"/>
 <contactref element="J9" pad="P$3_SLEEVE"/>
 <contactref element="J8" pad="P$3_SLEEVE"/>
@@
 <wire x1="35.18245" y1="26.7336" x2="55.3746" y2="26.7336" width="0.508" layer="16"/>
 </signal>
-<signal name="N$35">
-<contactref element="J6" pad="P$1_TIP"/>
-<contactref element="R18" pad="2"/>
-<contactref element="R19" pad="2"/>
-<contactref element="VOL" pad="2"/>
-<wire x1="20.955" y1="42.149" x2="20.955" y2="41.895" width="0.508" layer="1"/>
-<wire x1="20.955" y1="41.895" x2="13.081" y2="34.021" width="0.508" layer="1"/>
-<wire x1="13.081" y1="34.021" x2="13.081" y2="3.255" width="0.508" layer="1"/>
-<wire x1="16.51" y1="1.35" x2="14.986" y2="1.35" width="0.508" layer="1"/>
-<wire x1="14.986" y1="1.35" x2="13.081" y2="3.255" width="0.508" layer="1"/>
-<wire x1="49.215" y1="35.814" x2="49.215" y2="32.639" width="0.508" layer="16"/>
-<wire x1="49.215" y1="35.814" x2="49.215" y2="34.29" width="0.508" layer="16"/>
-<wire x1="49.215" y1="34.29" x2="28.814" y2="34.29" width="0.508" layer="16"/>
-<wire x1="28.814" y1="34.29" x2="20.955" y2="42.149" width="0.508" layer="16"/>
-</signal>
 <signal name="N$36">
-<contactref element="R19" pad="1"/>
 <contactref element="PAN" pad="3"/>
 <contactref element="R21" pad="2"/>
-<wire x1="51.115" y1="29.718" x2="51.115" y2="32.639" width="0.508" layer="16"/>
-<wire x1="52.665" y1="42.149" x2="52.705" y2="42.109" width="0.508" layer="16"/>
-<wire x1="52.705" y1="42.109" x2="52.705" y2="33.655" width="0.508" layer="16"/>
-<wire x1="52.705" y1="33.655" x2="51.689" y2="32.639" width="0.508" layer="16"/>
-<wire x1="51.689" y1="32.639" x2="51.115" y2="32.639" width="0.508" layer="16"/>
+<wire x1="52.665" y1="42.149" x2="52.665" y2="39.899" width="0.508" layer="16"/>
+<wire x1="52.665" y1="39.899" x2="52.451" y2="39.685" width="0.508" layer="16"/>
 </signal>
 <signal name="N$38">
-<contactref element="R18" pad="1"/>
 <contactref element="PAN" pad="1"/>
 <contactref element="R20" pad="2"/>
-<wire x1="51.115" y1="35.814" x2="51.115" y2="38.735" width="0.508" layer="16"/>
-<wire x1="47.665" y1="42.149" x2="47.665" y2="41.235" width="0.508" layer="16"/>
-<wire x1="47.665" y1="41.235" x2="48.26" y2="40.64" width="0.508" layer="16"/>
-<wire x1="48.26" y1="40.64" x2="50.165" y2="40.64" width="0.508" layer="16"/>
-<wire x1="50.165" y1="40.64" x2="51.115" y2="39.69" width="0.508" layer="16"/>
-<wire x1="51.115" y1="39.69" x2="51.115" y2="38.735" width="0.508" layer="16"/>
+<wire x1="47.665" y1="42.149" x2="47.665" y2="39.852" width="0.508" layer="16"/>
+<wire x1="47.665" y1="39.852" x2="47.498" y2="39.685" width="0.508" layer="16"/>
 </signal>
 <signal name="SV1">
@@
 <wire x1="8.636" y1="25.654" x2="19.304" y2="25.654" width="0.508" layer="16"/>
 <via x="27.178" y="33.528" extent="1-16" drill="0.35"/>
-<via x="28.956" y="35.306" extent="1-16" drill="0.35"/>
-<wire x1="28.956" y1="35.306" x2="27.178" y2="33.528" width="0.508" layer="1"/>
-<wire x1="45.6466" y1="35.1666" x2="49.215" y2="38.735" width="0.508" layer="16"/>
-<wire x1="28.956" y1="35.306" x2="29.0954" y2="35.1666" width="0.508" layer="16"/>
-<wire x1="45.6466" y1="35.1666" x2="29.0954" y2="35.1666" width="0.508" layer="16"/>
+<via x="29.337" y="35.687" extent="1-16" drill="0.35"/>
+<wire x1="29.337" y1="35.687" x2="27.178" y2="33.528" width="0.508" layer="1"/>
+<wire x1="46.095590625" y1="35.8016" x2="47.498" y2="37.785" width="0.508" layer="16"/>
+<wire x1="46.095590625" y1="35.8016" x2="29.4516" y2="35.8016" width="0.508" layer="16"/>
+<wire x1="29.337" y1="35.687" x2="29.4516" y2="35.8016" width="0.508" layer="16"/>
 </signal>
 <signal name="N$43">
@@
 <wire x1="4.318" y1="24.40403125" x2="5.83993125" y2="22.8821" width="0.508" layer="1"/>
 <via x="11.938" y="22.86" extent="1-16" drill="0.35"/>
-<wire x1="45.212" y1="22.86" x2="11.938" y2="22.86" width="0.508" layer="16"/>
-<wire x1="45.212" y1="22.86" x2="46.482" y2="24.13" width="0.508" layer="16"/>
-<via x="46.482" y="24.13" extent="1-16" drill="0.35"/>
-<via x="46.482" y="28.194" extent="1-16" drill="0.35"/>
-<wire x1="48.453" y1="29.68844375" x2="47.99075" y2="29.70275" width="0.508" layer="16"/>
-<wire x1="47.99075" y1="29.70275" x2="46.482" y2="28.194" width="0.508" layer="16"/>
-<wire x1="49.215" y1="29.718" x2="48.453" y2="29.718" width="0.508" layer="16"/>
-<wire x1="48.453" y1="29.718" x2="48.453" y2="29.68844375" width="0.508" layer="16"/>
-<wire x1="46.482" y1="28.194" x2="46.482" y2="24.13" width="0.508" layer="1"/>
+<wire x1="51.562" y1="22.86" x2="11.938" y2="22.86" width="0.508" layer="16"/>
+<wire x1="51.562" y1="22.86" x2="52.578" y2="23.876" width="0.508" layer="16"/>
+<via x="52.578" y="23.876" extent="1-16" drill="0.35"/>
+<via x="52.578" y="28.194" extent="1-16" drill="0.35"/>
+<wire x1="52.578" y1="23.876" x2="52.578" y2="28.194" width="0.508" layer="1"/>
+<wire x1="52.451" y1="37.785" x2="52.451" y2="28.321" width="0.508" layer="16"/>
+<wire x1="52.451" y1="28.321" x2="52.578" y2="28.194" width="0.508" layer="16"/>
 </signal>
 <signal name="N$32">
@@
 <wire x1="36.86" y1="48.925" x2="36.86" y2="47.5" width="1.016" layer="16"/>
 </signal>
+<signal name="N$34">
+<contactref element="VOL" pad="2"/>
+<contactref element="PAN" pad="2"/>
+<contactref element="J6" pad="P$1_TIP"/>
+<wire x1="20.955" y1="42.149" x2="13.081" y2="34.275" width="0.508" layer="1"/>
+<wire x1="13.081" y1="34.275" x2="13.081" y2="3.255" width="0.508" layer="1"/>
+<wire x1="16.51" y1="1.35" x2="14.986" y2="1.35" width="0.508" layer="1"/>
+<wire x1="14.986" y1="1.35" x2="13.081" y2="3.255" width="0.508" layer="1"/>
+<wire x1="50.165" y1="42.149" x2="50.2284" y2="42.0856" width="0.508" layer="16"/>
+<wire x1="50.2284" y1="42.0856" x2="50.2284" y2="36.2046625" width="0.508" layer="16"/>
+<wire x1="28.19813125" y1="34.9024" x2="20.955" y2="42.14553125" width="0.508" layer="16"/>
+<wire x1="20.955" y1="42.149" x2="20.955" y2="42.14553125" width="0.508" layer="16"/>
+<wire x1="28.19813125" y1="34.9024" x2="48.9261375" y2="34.9024" width="0.508" layer="16"/>
+<wire x1="48.9261375" y1="34.9024" x2="50.2284" y2="36.2046625" width="0.508" layer="16"/>
+</signal>
 </signals>
