File: PANS.sch (EAGLE design)
At the start: 69 parts, among them IC1 TL074, IC2 TL074, J1 THONKICONNNEW, J15 power, J2 THONKICONNNEW, J3 THONKICONNNEW, J4 THONKICONNNEW, J5 THONKICONNNEW, J6 THONKICONNNEW, J7 Stereo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

Commit message: Add files via upload
Parts:
- removed R18, R19: 1K, resistor:R-US_M0805
- PAN: value 10K -> B1M
Connections:
- removed net N$35: J6.TIP, R18.2, R19.2, VOL.S
- new net N$34: J6.TIP, PAN.S, VOL.S
- net GND: no longer PAN.S
- net N$36: no longer R19.1
- net N$38: no longer R18.1
Other:
- moved on the sheet: PAN
Changed lines of the file:
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@@
 <part name="2VOL" library="MusicThingModular" deviceset="9MM_SNAP-IN_POT" device="_" value="1MA"/>
 <part name="1VOL" library="MusicThingModular" deviceset="9MM_SNAP-IN_POT" device="_" value="1MA"/>
-<part name="PAN" library="MusicThingModular" deviceset="9MM_SNAP-IN_POT" device="_" value="10K"/>
+<part name="PAN" library="MusicThingModular" deviceset="9MM_SNAP-IN_POT" device="_" value="B1M"/>
 <part name="IC2" library="MusicThingModular" deviceset="TL074" device="_SMD" value="TL074"/>
 <part name="J8" library="MusicThingModular" deviceset="THONKICONN" device="NEW" value="THONKICONNNEW"/>
@@
 <part name="SUPPLY23" library="supply2" deviceset="GND" device=""/>
 <part name="R21" library="resistor" deviceset="R-US_" device="M0805" value="1K"/>
-<part name="R18" library="resistor" deviceset="R-US_" device="M0805" value="1K"/>
-<part name="R19" library="resistor" deviceset="R-US_" device="M0805" value="1K"/>
-<part name="SUPPLY25" library="supply2" deviceset="GND" device=""/>
 <part name="SUPPLY26" library="supply2" deviceset="GND" device=""/>
 <part name="SUPPLY27" library="supply2" deviceset="GND" device=""/>
@@
 <attribute name="VALUE" x="50.8" y="121.92" size="1.778" layer="96" rot="MR180"/>
 </instance>
-<instance part="PAN" gate="G$1" x="170.18" y="58.42" smashed="yes" rot="R270">
-<attribute name="NAME" x="167.64" y="63.5" size="1.778" layer="95"/>
-<attribute name="VALUE" x="167.64" y="60.96" size="1.778" layer="96"/>
+<instance part="PAN" gate="G$1" x="170.18" y="58.42" smashed="yes" rot="MR90">
+<attribute name="NAME" x="167.64" y="53.34" size="1.778" layer="95" rot="MR180"/>
+<attribute name="VALUE" x="167.64" y="55.88" size="1.778" layer="96" rot="MR180"/>
 </instance>
 <instance part="IC2" gate="A" x="86.36" y="101.6" smashed="yes">
@@
 <attribute name="NAME" x="176.3014" y="44.45" size="1.778" layer="95" rot="R90"/>
 <attribute name="VALUE" x="181.102" y="44.45" size="1.778" layer="96" rot="R90"/>
-</instance>
-<instance part="R18" gate="G$1" x="162.56" y="68.58" smashed="yes" rot="R90">
-<attribute name="NAME" x="161.0614" y="64.77" size="1.778" layer="95" rot="R90"/>
-<attribute name="VALUE" x="165.862" y="64.77" size="1.778" layer="96" rot="R90"/>
-</instance>
-<instance part="R19" gate="G$1" x="177.8" y="68.58" smashed="yes" rot="R90">
-<attribute name="NAME" x="176.3014" y="64.77" size="1.778" layer="95" rot="R90"/>
-<attribute name="VALUE" x="181.102" y="64.77" size="1.778" layer="96" rot="R90"/>
-</instance>
-<instance part="SUPPLY25" gate="GND" x="170.18" y="50.8" smashed="yes">
-<attribute name="VALUE" x="168.275" y="47.625" size="1.778" layer="96"/>
 </instance>
 <instance part="SUPPLY26" gate="GND" x="190.5" y="33.02" smashed="yes">
@@
 <pinref part="J6" gate="G$1" pin="SLEEVE"/>
 <pinref part="SUPPLY23" gate="GND" pin="GND"/>
-</segment>
-<segment>
-<pinref part="PAN" gate="G$1" pin="S"/>
-<pinref part="SUPPLY25" gate="GND" pin="GND"/>
 </segment>
 <segment>
@@
 </segment>
 </net>
-<net name="N$35" class="0">
-<segment>
-<pinref part="J6" gate="G$1" pin="TIP"/>
-<wire x1="190.5" y1="88.9" x2="177.8" y2="88.9" width="0.1524" layer="91"/>
-<wire x1="177.8" y1="88.9" x2="177.8" y2="73.66" width="0.1524" layer="91"/>
-<pinref part="R18" gate="G$1" pin="2"/>
-<wire x1="162.56" y1="73.66" x2="177.8" y2="73.66" width="0.1524" layer="91"/>
-<pinref part="R19" gate="G$1" pin="2"/>
-<junction x="177.8" y="73.66"/>
-<junction x="177.8" y="73.66"/>
-<pinref part="VOL" gate="G$1" pin="S"/>
-<wire x1="162.56" y1="76.2" x2="162.56" y2="73.66" width="0.1524" layer="91"/>
-<junction x="162.56" y="73.66"/>
-<junction x="177.8" y="73.66"/>
-</segment>
-</net>
 <net name="N$36" class="0">
 <segment>
-<pinref part="R19" gate="G$1" pin="1"/>
-<wire x1="177.8" y1="63.5" x2="177.8" y2="58.42" width="0.1524" layer="91"/>
 <pinref part="PAN" gate="G$1" pin="E"/>
 <pinref part="R21" gate="G$1" pin="2"/>
 <wire x1="177.8" y1="53.34" x2="177.8" y2="58.42" width="0.1524" layer="91"/>
-<junction x="177.8" y="58.42"/>
 </segment>
 </net>
 <net name="N$38" class="0">
 <segment>
-<pinref part="R18" gate="G$1" pin="1"/>
-<wire x1="162.56" y1="63.5" x2="162.56" y2="58.42" width="0.1524" layer="91"/>
 <pinref part="PAN" gate="G$1" pin="A"/>
 <pinref part="R20" gate="G$1" pin="2"/>
 <wire x1="162.56" y1="53.34" x2="162.56" y2="58.42" width="0.1524" layer="91"/>
-<junction x="162.56" y="58.42"/>
 </segment>
 </net>
@@
 </segment>
 </net>
+<net name="N$34" class="0">
+<segment>
+<pinref part="VOL" gate="G$1" pin="S"/>
+<wire x1="162.56" y1="76.2" x2="162.56" y2="67.31" width="0.1524" layer="91"/>
+<wire x1="162.56" y1="67.31" x2="170.18" y2="67.31" width="0.1524" layer="91"/>
+<pinref part="PAN" gate="G$1" pin="S"/>
+<wire x1="170.18" y1="67.31" x2="170.18" y2="63.5" width="0.1524" layer="91"/>
+<wire x1="170.18" y1="67.31" x2="177.8" y2="67.31" width="0.1524" layer="91"/>
+<junction x="170.18" y="67.31"/>
+<pinref part="J6" gate="G$1" pin="TIP"/>
+<wire x1="190.5" y1="88.9" x2="177.8" y2="88.9" width="0.1524" layer="91"/>
+<wire x1="177.8" y1="88.9" x2="177.8" y2="67.31" width="0.1524" layer="91"/>
+</segment>
+</net>
